File: pcb/flinx.kicad_pcb (KiCad board)
At the start: 4 copper layers, 252.5 x 68.8 mm, 139 parts, among them J1 USB_C_Receptacle_USB2.0_14P, SW1 SW_Push, SW10 SW_Push, SW11 SW_Push, SW12 SW_Push, SW13 SW_Push, SW14 SW_Push, SW15 SW_Push, SW16 SW_Push, SW17 SW_Push, SW18 SW_Push, SW19 SW_Push, SW2 SW_Push, SW20 SW_Push, SW21 SW_Push, SW22 SW_Push, SW23 SW_Push, SW24 SW_Push, SW25 SW_Push, SW26 SW_Push, SW27 SW_Push, SW28 SW_Push, SW29 SW_Push, SW3 SW_Push, SW30 SW_Push, SW31 SW_Push, SW32 SW_Push, SW33 SW_Push, SW34 SW_Push, SW35 SW_Push, SW36 SW_Push, SW37 SW_Push, SW38 SW_Push, SW39 SW_Push, SW4 SW_Push, SW40 SW_Push, SW41 SW_Push, SW42 SW_Push, SW43 SW_Push, SW44 SW_Push, SW45 SW_Push, SW46 SW_Push, SW47 SW_Push, SW48 SW_Push, SW49 SW_SPDT, SW5 SW_Push, SW6 SW_Push, SW7 SW_Push, SW8 SW_Push, SW9 SW_Push, U1 nRF52833_QDxx, U2 TP4057, Y1 32MHz

Commit message: Update PCB
Parts:
- added REF**: Drill_3.5x3.5, Project:Drill_3.5x3.5, F.Cu at (87.5, 116.7)
- added REF**: Drill_3.5x3.5, Project:Drill_3.5x3.5, F.Cu at (246.2, 82.7)
- added REF**: Drill_3.5x3.5, Project:Drill_3.5x3.5, F.Cu at (50.4, 99.7)
- added REF**: Drill_3.5x3.5, Project:Drill_3.5x3.5, F.Cu at (209.1, 116.7)
- L1, L3, L4: value 4.7nH -> 4.7 nH
- L2: value 2.2nH -> 2.2 nH
- L5: value 2.7nH -> 2.7 nH
- L6: value 3.3nH -> 3.3 nH
- Y1: footprint Crystal:Crystal_SMD_MicroCrystal_CC7V-T1A-2Pin_3.2x1.5mm -> Crystal:Crystal_SMD_SeikoEpson_FA128-4Pin_2.0x1.6mm
- moved R1 0.62 mm to (251.2, 78.5)
- moved R2 0.62 mm to (251.2, 80.3)
- moved R3 0.62 mm to (251.2, 76.3)
- moved R4 0.62 mm to (251.2, 82.5)
- moved Y1 0.59 mm to (141.8, 121.5)
Connections:
- Y1 pad 2: Net-(U1-XC2) -> GND
Routing:
- net GND: track 13.8 -> 15.7 mm
- net Net-(U1-XC1): track 11.2 -> 12.3 mm
- net C4: track 147.9 -> 148.8 mm
- net Net-(U1-XC2): track 8.41 -> 7.64 mm
- net Net-(J1-D+-PadA6): track 18.3 -> 17.7 mm
- net Net-(J1-CC2): track 18.9 -> 18.3 mm
- net Net-(J1-CC1): track 16.8 -> 16.1 mm
- net Net-(J1-D--PadA7): track 19.7 -> 19.1 mm

Commit message: Swap to BL654
Parts:
- removed AE1: Antenna, RF_Antenna:Johanson_2450AT18x100
- removed C10: 100 pF, Capacitor_SMD:C_0603_1608Metric
- removed C11, C16, C17, C18: 100 nF, Capacitor_SMD:C_0603_1608Metric
- removed C14: 1.2 pF, Capacitor_SMD:C_0603_1608Metric
- removed C15, C7, C8, C9: 4.7 uF, Capacitor_SMD:C_0603_1608Metric
- removed the C5 at (150.6, 122.0)
- removed the C6 at (154.8, 119.5)
- removed L1, L3, L4: 4.7 nH, Inductor_SMD:L_0603_1608Metric
- removed L2: 2.2 nH, Inductor_SMD:L_0603_1608Metric
- removed L5: 2.7 nH, Inductor_SMD:L_0603_1608Metric
- removed L6: 3.3 nH, Inductor_SMD:L_0603_1608Metric
- removed TP5: TestPoint, Project:Pad_SMD_1.5x1.5
- removed the U1 at (148.2, 115.7)
- added ANT1: 451-00001, Project:45100001, B.Cu at (148.3, 117.5)
- C2: value 12 pF -> 10 pF
- C3: value 4.7 uF -> 100 nF
- C4: value 4.7 uF -> 10 uF
- Y1: value 32MHz -> 32.768 kHz 9 pF; footprint Crystal:Crystal_SMD_SeikoEpson_FA128-4Pin_2.0x1.6mm -> Crystal:Crystal_SMD_MicroCrystal_CC7V-T1A-2Pin_3.2x1.5mm_HandSoldering
- moved Y1 39.2 mm to (180.9, 119.5), turned to 180 degrees
- moved C1 36.2 mm to (182.5, 122.5)
- moved C2 34.7 mm to (179.2, 122.5)
- moved C4 5.37 mm to (159.2, 111.0), turned to 180 degrees
- moved D41 5.00 mm to (137.6, 116.9)
- moved C3 4.48 mm to (159.2, 113.0), turned to 180 degrees
- renumbered C12 to C5, C13 to C6, U2 to U1
Connections:
- net Net-(U1-XC1) renamed XL1
- C2 pad 1: Net-(U1-XC2) -> XL2
- C4 pad 1: VBUS -> VDDH
- TP1 pad 1: nRF -> GND
- TP2 pad 1: GND -> RESET
- TP3 pad 1: RESET -> SWCLK
- TP4 pad 1: SWCLK -> SWDIO
- Y1 pad 2: GND -> XL2
Routing:
- net nRF: track 110.0 -> 29.5 mm, vias 8 -> 2
- net XL2: track 0.00 -> 43.3 mm, vias 0 -> 2
- net XL1: track 12.3 -> 47.7 mm, vias 0 -> 2
- net C8: track 131.7 -> 101.9 mm
- net RF: track 22.3 -> 0.00 mm
- net DEC4: track 20.1 -> 0.00 mm, vias 2 -> 0
- net C7: track 87.7 -> 74.8 mm, vias 5 -> 4
- net C6: track 79.6 -> 68.3 mm
- net Net-(U1-ANT): track 9.82 -> 0.00 mm
- net Net-(C6-Pad1): track 9.45 -> 0.00 mm
- net Net-(U1-XC2): track 7.64 -> 0.00 mm
- net VBUS: track 186.8 -> 179.5 mm, vias 4 -> 3
- net Net-(U1-DEC3): track 7.16 -> 0.00 mm
- net Net-(U1-DEC1): track 6.84 -> 0.00 mm
- net C10: track 183.9 -> 190.3 mm, vias 5 -> 6
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- removed copper zone on In1.Cu, net GND
Other:
- board text added: "BATT+"
- board text added: "BATT-"

Commit message: Move decoupling caps
Parts:
- moved C3 3.35 mm to (157.7, 110.0)
- moved C4 1.95 mm to (157.8, 112.2)
Connections:
- C3 pad 1: VDDH -> GND
- C3 pad 2: GND -> VDDH
- C4 pad 1: VDDH -> GND
- C4 pad 2: GND -> VDDH
Routing:
- net R4: track 322.3 -> 323.1 mm
- net VDDH: vias 3 -> 4

Commit message: Update value
Parts:
- R6: value 75k -> 10k
Changed lines of the file:
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@@
 			(outputformat 1)
 			(mirror no)
-			(drillshape 1)
+			(drillshape 0)
 			(scaleselection 1)
 			(outputdirectory "")
@@
 			)
 		)
-		(property "Value" "75k"
+		(property "Value" "10k"
 			(at 0 -1.43 0)
 			(layer "B.Fab")

Commit message: Add logo
Parts:
- added G***: LOGO, LOGO, F.Cu at (117.0, 116.7)
